Commit message: fix error

File: URDFoptimizer/render/mobility.urdf (robot description, URDF)
Before this commit: robot partnet_10798ccb7072393e86d53ab0fe94e911, 3 links, 2 joints
Links:
- link link_0: geometry collision mesh filename=glb/part_0_geometry_0.glb; visual mesh filename=glb/part_0_geometry_0.glb
- link link_1: geometry collision mesh filename=glb/part_1_geometry_1.glb; visual mesh filename=glb/part_1_geometry_1.glb
