Commit message: fix error

File: URDFoptimizer/input/mobility.urdf (robot description, URDF)
Before this commit: robot partnet_10798ccb7072393e86d53ab0fe94e911, 3 links, 2 joints
Links:
- link link_0: geometry collision mesh filename=glb/part_0_geometry_0.glb; visual mesh filename=glb/part_0_geometry_0.glb
- link link_1: geometry collision mesh filename=glb/part_1_geometry_1.glb; visual mesh filename=glb/part_1_geometry_1.glb

File: URDFoptimizer/input/mobility_optimized.urdf (robot description, URDF)
Before this commit: robot partnet_10798ccb7072393e86d53ab0fe94e911, 3 links, 2 joints
Links:
- link link_0: geometry collision mesh filename=glb/part_0_geometry_0.glb; visual mesh filename=glb/part_0_geometry_0.glb
- link link_1: geometry collision mesh filename=glb/part_1_geometry_1.glb; visual mesh filename=glb/part_1_geometry_1.glb
Joints:
- joint joint_0: origin xyz=0.18202803 0.00000000 0.20976162 -> xyz=-0.37604299 0.07863900 0.51754802
